Commit message: urdf new contact frames & xml friction coefficient

File: resources/description_files/urdf/go2/go2.urdf (robot description, URDF)
Before this commit: robot go2_description, 43 links, 42 joints
Links:
- added link FL_foot_
- added link FR_foot_
- added link RL_foot_
- added link RR_foot_
Joints:
- added joint FL_foot_joint_: type fixed, parent FL_calflower1, child FL_foot_, origin xyz=0.005 0 -0.05 rpy=0 0 0
- added joint FR_foot_joint_: type fixed, parent FR_calflower1, child FR_foot_, origin xyz=0.005 0 -0.05 rpy=0 0 0
- added joint RL_foot_joint_: type fixed, parent RL_calflower1, child RL_foot_, origin xyz=0.005 0 -0.05 rpy=0 0 0
- added joint RR_foot_joint_: type fixed, parent RR_calflower1, child RR_foot_, origin xyz=0.005 0 -0.05 rpy=0 0 0
