Commit message: added: lidar working

File: resources/description_files/urdf/go2/go2_gz.urdf (robot description, URDF)
Before this commit: robot go2_description, 42 links, 41 joints
Links:
- link utlidar_lidar: mass 0 -> 0.001
Joints:
- joint radar_joint: axis 0 0 0 -> (none); origin xyz=0.28945 0 -0.046825 rpy=0 2.8782 0 -> xyz=0.28945 0 0.1 rpy=0 0 0; parent base -> Head_lower

Commit message: fix: polish gazebo code

File: resources/description_files/urdf/go2/go2_gz.urdf (robot description, URDF)
Before this commit: robot go2_description, 42 links, 41 joints
Links:
- link utlidar_lidar: mass 0.001 -> 0
Joints:
- joint radar_joint: axis (none) -> 0 0 0; origin xyz=0.28945 0 0.1 rpy=0 0 0 -> xyz=0.28945 0 -0.046825 rpy=0 2.8782 0; parent Head_lower -> base

Commit message: fixed: lidar configuration + walk upstairs

File: resources/description_files/urdf/go2/go2_gz.urdf (robot description, URDF)
Before this commit: robot go2_description, 42 links, 41 joints
Links:
- link utlidar_lidar: mass 0 -> 0.03; geometry collision cylinder length=0.04 radius=0.03

Commit message: fixed: MAJOR ISSUE git add .! The utlidar_lidar link needed to be shift down (z=-0.47->z=0.49) to avoid self-collision)

File: resources/description_files/urdf/go2/go2_gz.urdf (robot description, URDF)
Before this commit: robot go2_description, 42 links, 41 joints
Joints:
- joint radar_joint: origin xyz=0.28945 0 -0.046825 rpy=0 2.8782 0 -> xyz=0.28945 0 -0.049 rpy=0 2.8782 0
