Commit message: Add G1 with grippers, awaiting gripper simulation

File: resources/description_files/urdf/g1/g1_29dof_dx3.urdf (robot description, URDF)
Before this commit: robot g1_29dof_with_hand_rev_1_0, 53 links, 52 joints
Links:
- link head_link: geometry collision mesh filename=package://huro/resources/description_files/meshes/g1/head_l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; visual mesh filename=package://huro/resources/description_files/meshes/g1/head_l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
- link left_ankle_pitch_link: geometry collision mesh filename=package://huro/resources/description_files/meshes/g1/left_a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; visual mesh filename=package://huro/resources/description_files/meshes/g1/left_a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
- link left_ankle_roll_link: geometry collision sphere radius=0.005; collision sphere radius=0.005
- link left_elbow_link: geometry collision mesh filename=package://huro/resources/description_files/meshes/g1/left_e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; visual mesh filename=package://huro/resources/description_files/meshes/g1/left_e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
- link left_hand_index_0_link: geometry collision mesh filename=package://huro/resources/description_files/meshes/g1/left_h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; visual mesh filename=package://huro/resources/description_files/meshes/g1/left_h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
- link left_hand_index_1_link: geometry collision mesh filename=package://huro/resources/description_files/meshes/g1/left_h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; visual mesh filename=package://huro/resources/description_files/meshes/g1/left_h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
- link left_hand_middle_0_link: geometry collision mesh filename=package://huro/resources/description_files/meshes/g1/left_h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; visual mesh filename=package://huro/resources/description_files/meshes/g1/left_h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
- link left_hand_middle_1_link: geometry collision mesh filename=package://huro/resources/description_files/meshes/g1/left_h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; visual mesh filename=package://huro/resources/description_files/meshes/g1/left_h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
- link left_hand_palm_link: geometry collision mesh filename=package://huro/resources/description_files/meshes/g1/left_h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; visual mesh filename=package://huro/resources/description_files/meshes/g1/left_h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
- link left_hand_thumb_0_link: geometry collision mesh filename=package://huro/resources/description_files/meshes/g1/left_h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; visual mesh filename=package://huro/resources/description_files/meshes/g1/left_h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
- link left_hand_thumb_1_link: geometry collision box size=0.02 0.03 0.02; visual mesh filename=package://huro/resources/description_files/meshes/g1/left_h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
- link left_hand_thumb_2_link: geometry collision mesh filename=package://huro/resources/description_files/meshes/g1/left_h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; visual mesh filename=package://huro/resources/description_files/meshes/g1/left_h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
- link left_hip_pitch_link: geometry collision mesh filename=package://huro/resources/description_files/meshes/g1/left_h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; visual mesh filename=package://huro/resources/description_files/meshes/g1/left_h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
- link left_hip_roll_link: geometry collision mesh filename=package://huro/resources/description_files/meshes/g1/left_h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; visual mesh filename=package://huro/resources/description_files/meshes/g1/left_h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
- link left_hip_yaw_link: geometry collision mesh filename=package://huro/resources/description_files/meshes/g1/left_h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; visual mesh filename=package://huro/resources/description_files/meshes/g1/left_h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
- link left_knee_link: geometry collision mesh filename=package://huro/resources/description_files/meshes/g1/left_k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; visual mesh filename=package://huro/resources/description_files/meshes/g1/left_k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
- link left_shoulder_pitch_link: geometry collision cylinder length=0.05 radius=0.03; visual mesh filename=package://huro/resources/description_files/meshes/g1/left_s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
- link left_shoulder_roll_link: geometry collision cylinder length=0.03 radius=0.03; visual mesh filename=package://huro/resources/description_files/meshes/g1/left_s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
- link left_shoulder_yaw_link: geometry collision mesh filename=package://huro/resources/description_files/meshes/g1/left_s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; visual mesh filename=package://huro/resources/description_files/meshes/g1/left_s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
- link left_wrist_pitch_link: geometry collision mesh filename=package://huro/resources/description_files/meshes/g1/left_w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; visual mesh filename=package://huro/resources/description_files/meshes/g1/left_w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
- link left_wrist_roll_link: geometry collision mesh filename=package://huro/resources/description_files/meshes/g1/left_w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; visual mesh filename=package://huro/resources/description_files/meshes/g1/left_w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
- link left_wrist_yaw_link: geometry collision mesh filename=package://huro/resources/description_files/meshes/g1/left_w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; visual mesh filename=package://huro/resources/description_files/meshes/g1/left_w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
- link logo_link: geometry collision mesh filename=package://huro/resources/description_files/meshes/g1/logo_l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; visual mesh filename=package://huro/resources/description_files/meshes/g1/logo_l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
- link pelvis: geometry visual mesh filename=package://huro/resources/description_files/meshes/g1/pelvis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
- link pelvis_contour_link: geometry collision mesh filename=package://huro/resources/description_files/meshes/g1/pelvis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; visual mesh filename=package://huro/resources/description_files/meshes/g1/pelvis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
- link right_ankle_pitch_link: geometry collision mesh filename=package://huro/resources/description_files/meshes/g1/right_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; visual mesh filename=package://huro/resources/description_files/meshes/g1/right_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
- link right_ankle_roll_link: geometry collision sphere radius=0.005; collision sphere radius=0.005
- link right_elbow_link: geometry collision mesh filename=package://huro/resources/description_files/meshes/g1/right_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; visual mesh filename=package://huro/resources/description_files/meshes/g1/right_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
- link right_hand_index_0_link: geometry collision mesh filename=package://huro/resources/description_files/meshes/g1/right_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; visual mesh filename=package://huro/resources/description_files/meshes/g1/right_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
- link right_hand_index_1_link: geometry collision mesh filename=package://huro/resources/description_files/meshes/g1/right_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; visual mesh filename=package://huro/resources/description_files/meshes/g1/right_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
- link right_hand_middle_0_link: geometry collision mesh filename=package://huro/resources/description_files/meshes/g1/right_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; visual mesh filename=package://huro/resources/description_files/meshes/g1/right_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
- link right_hand_middle_1_link: geometry collision mesh filename=package://huro/resources/description_files/meshes/g1/right_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; visual mesh filename=package://huro/resources/description_files/meshes/g1/right_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
- link right_hand_palm_link: geometry collision mesh filename=package://huro/resources/description_files/meshes/g1/right_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; visual mesh filename=package://huro/resources/description_files/meshes/g1/right_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
- link right_hand_thumb_0_link: geometry collision mesh filename=package://huro/resources/description_files/meshes/g1/right_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; visual mesh filename=package://huro/resources/description_files/meshes/g1/right_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
- link right_hand_thumb_1_link: geometry collision box size=0.02 0.03 0.02; visual mesh filename=package://huro/resources/description_files/meshes/g1/right_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
- link right_hand_thumb_2_link: geometry collision mesh filename=package://huro/resources/description_files/meshes/g1/right_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; visual mesh filename=package://huro/resources/description_files/meshes/g1/right_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
- link right_hip_pitch_link: geometry collision mesh filename=package://huro/resources/description_files/meshes/g1/right_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; visual mesh filename=package://huro/resources/description_files/meshes/g1/right_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
- link right_hip_roll_link: geometry collision mesh filename=package://huro/resources/description_files/meshes/g1/right_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; visual mesh filename=package://huro/resources/description_files/meshes/g1/right_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
- link right_hip_yaw_link: geometry collision mesh filename=package://huro/resources/description_files/meshes/g1/right_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; visual mesh filename=package://huro/resources/description_files/meshes/g1/right_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
- link right_knee_link: geometry collision mesh filename=package://huro/resources/description_files/meshes/g1/right_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; visual mesh filename=package://huro/resources/description_files/meshes/g1/right_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
- link right_shoulder_pitch_link: geometry collision cylinder length=0.05 radius=0.03; visual mesh filename=package://huro/resources/description_files/meshes/g1/right_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
- link right_shoulder_roll_link: geometry collision cylinder length=0.03 radius=0.03; visual mesh filename=package://huro/resources/description_files/meshes/g1/right_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
- link right_shoulder_yaw_link: geometry collision mesh filename=package://huro/resources/description_files/meshes/g1/right_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; visual mesh filename=package://huro/resources/description_files/meshes/g1/right_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
- link right_wrist_pitch_link: geometry collision mesh filename=package://huro/resources/description_files/meshes/g1/right_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; visual mesh filename=package://huro/resources/description_files/meshes/g1/right_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
- link right_wrist_roll_link: geometry collision mesh filename=package://huro/resources/description_files/meshes/g1/right_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; visual mesh filename=package://huro/resources/description_files/meshes/g1/right_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
- link right_wrist_yaw_link: geometry collision mesh filename=package://huro/resources/description_files/meshes/g1/right_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; visual mesh filename=package://huro/resources/description_files/meshes/g1/right_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
- link torso_link: geometry collision mesh filename=package://huro/resources/description_files/meshes/g1/torso_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; visual mesh filename=package://huro/resources/description_files/meshes/g1/torso_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
- link waist_roll_link: geometry visual mesh filename=package://huro/resources/description_files/meshes/g1/waist_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
- link waist_yaw_link: geometry visual mesh filename=package://huro/resources/description_files/meshes/g1/waist_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
