Commit message: Add custom head ref frame in G1 urdf

File: resources/description_files/urdf/g1/g1_29dof.urdf (robot description, URDF)
Before this commit: robot g1_29dof_rev_1_0, 57 links, 56 joints
Links:
- added link head_custom_link
Joints:
- added joint head_custom_fix_joint: type fixed, parent imu_in_torso, child head_custom_link, origin xyz=0.05 0.0 0.2 rpy=0 0 0
